File: hardware/LoRa Ground Station.kicad_pcb (KiCad board)
At the start: 4 copper layers, 33 x 44 mm, 51 parts, among them J1 RFPC-SMA28-F, J2 USB_C_Receptacle_USB2.0_14P, SW1 BOOT, SW2 RESET, U1 RP2040, U2 SX1262IMLTRT, U3 PE4259, U4 AP2112K-3.3, U5 W25Q128JVS, Y1 ECS-TXO-25CSMV-320-DY-TR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

Commit message: Add files via upload
Parts:
- added G***: LOGO, LOGO, F.Cu at (156.1, 74.0)
- added G***: LOGO, LOGO, B.Cu at (165.0, 57.0)
- added G***: LOGO, LOGO, B.Cu at (163.4, 57.2)
- added R9: 10k, Resistor_SMD:R_0402_1005Metric, F.Cu at (152.8, 53.7)
- added U6: TPD1E0B04DPLR, footprints3:DPL0002A-MFG, F.Cu at (173.1, 74.7)
- C25, C26: value 3.3 pF -> 10 uF; footprint Capacitor_SMD:C_0402_1005Metric -> Capacitor_SMD:C_0603_1608Metric
- R5: value 27.3 -> 10k
- moved C22 10.6 mm to (160.8, 61.7), turned to -90 degrees
- moved R3 4.83 mm to (164.7, 48.9)
- moved R4 4.76 mm to (163.6, 48.9)
- moved C14 1.98 mm to (162.2, 52.0)
- moved R2 1.79 mm to (158.6, 63.5)
- moved SW2 1.31 mm to (162.5, 66.2)
- moved R5 1.27 mm to (164.3, 62.3)
- moved C15 1.13 mm to (163.4, 52.9)
- moved C25 1.03 mm to (168.1, 54.4)
- moved C16 0.99 mm to (164.0, 53.9)
- moved C18 0.73 mm to (159.8, 62.5)
- moved C24 0.69 mm to (160.8, 51.5)
- moved U4 0.57 mm to (167.9, 51.6)
- moved C23 0.54 mm to (162.3, 51.0), turned to 0 degrees
- moved J1 0.49 mm to (172.9, 79.0)
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Routing:
- net Net-(U1-USB_DM): track 1.35 -> 7.76 mm
- net Net-(U1-USB_DP): track 1.43 -> 7.76 mm
- net /USB_D_P: track 9.47 -> 4.15 mm
- net /USB_D_N: track 9.21 -> 4.09 mm
- net /RUN: track 4.73 -> 8.59 mm, vias 0 -> 2
- net +1.1: track 10.8 -> 14.6 mm
- net VBUS: track 13.4 -> 16.1 mm
- net /XOUT: track 1.22 -> 3.05 mm
- net Earth: track 14.8 -> 16.0 mm, vias 227 -> 180
- net Net-(C13-Pad1): track 4.17 -> 3.06 mm
- net Net-(U6-1_IO): track 5.46 -> 6.03 mm
- net +3.3V: track 30.4 -> 30.7 mm, vias 14 -> 13
Other:
- board text added: "C23"
- board text added: "Darsh LoRa"
